File: PCB/ESPrinkler Retic PCB/Power IO.kicad_sch (KiCad schematic)
At the start: 32 parts, among them J6 Conn_01x04, Q1 AO3400A, Q2 AO3400A, U1 TPS5430DDA

Commit message: Continue PCB layout
Final placements and traces of components for first revision.
Parts:
- R1, R4, R9: value 300R -> 1.2k; Manufacturer P/N 0805W8F3000T5E -> 0805W8F1201T5E; Supplier P/N C17617 -> C17379
Changed lines of the file:
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@@
 			)
 		)
-		(property "Value" "300R"
+		(property "Value" "1.2k"
 			(at 247.015 65.405 0)
 			(effects
@@
 			)
 		)
-		(property "Manufacturer P/N" "0805W8F3000T5E"
+		(property "Manufacturer P/N" "0805W8F1201T5E"
 			(at 242.57 63.5 0)
 			(effects
@@
 			)
 		)
-		(property "Supplier P/N" "C17617"
+		(property "Supplier P/N" "C17379"
 			(at 242.57 63.5 0)
 			(effects
@@
 			)
 		)
-		(property "Value" "300R"
+		(property "Value" "1.2k"
 			(at 97.79 107.95 0)
 			(effects
@@
 			)
 		)
-		(property "Manufacturer P/N" "0805W8F3000T5E"
+		(property "Manufacturer P/N" "0805W8F1201T5E"
 			(at 93.98 107.95 0)
 			(effects
@@
 			)
 		)
-		(property "Supplier P/N" "C17617"
+		(property "Supplier P/N" "C17379"
 			(at 93.98 107.95 0)
 			(effects
@@
 			)
 		)
-		(property "Value" "300R"
+		(property "Value" "1.2k"
 			(at 40.64 107.95 0)
 			(effects
@@
 			)
 		)
-		(property "Manufacturer P/N" "0805W8F3000T5E"
+		(property "Manufacturer P/N" "0805W8F1201T5E"
 			(at 36.83 107.95 0)
 			(effects
@@
 			)
 		)
-		(property "Supplier P/N" "C17617"
+		(property "Supplier P/N" "C17379"
 			(at 36.83 107.95 0)
 			(effects
